File: _autosave-Kicad-Midi2CV2.kicad_pcb (KiCad board)
At the start: 2 copper layers, 100 x 100 mm, 100 parts, among them IC101 MCP4725module, IC102 MCP4725module, J101 Doepfer connector, J102 Vin 7-12v, J103 MIDI OUT, J104 Power Conn, J105 CV7 in, J106 Gate1, J107 MIDI IN, J108 CV6 in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

Commit message: Jumper fixes
Parts:
- added F101: Polyfuse, Fuse:Fuse_1206_3216Metric_Pad1.42x1.75mm_HandSolder, F.Cu at (130.0, 54.0)
- J115: footprint Connector_PinHeader_2.54mm:PinHeader_1x12_P2.54mm_Vertical -> Connector_PinHeader_2.54mm:PinHeader_1x11_P2.54mm_Vertical
- J116: footprint Connector_PinHeader_2.54mm:PinHeader_1x12_P2.54mm_Horizontal -> Connector_PinHeader_2.54mm:PinHeader_1x11_P2.54mm_Horizontal
- J117: footprint Connector_PinHeader_2.54mm:PinHeader_1x08_P2.54mm_Vertical -> Connector_PinHeader_2.54mm:PinHeader_1x09_P2.54mm_Vertical
- J118: footprint Connector_PinHeader_2.54mm:PinHeader_1x08_P2.54mm_Horizontal -> Connector_PinHeader_2.54mm:PinHeader_1x09_P2.54mm_Horizontal
- moved C104 174.6 mm to (67.4, 154.1)
- moved C107 174.6 mm to (73.7, 139.1)
- moved C111 174.6 mm to (73.1, 125.0)
- moved IC101 174.6 mm to (80.1, 122.5)
- moved IC102 174.6 mm to (80.1, 140.9)
- moved R104 174.6 mm to (67.1, 136.4)
- moved R105 174.6 mm to (62.9, 136.4)
- moved R106 174.6 mm to (76.3, 150.4)
- moved R107 174.6 mm to (76.3, 146.6)
- moved R112 174.6 mm to (66.7, 130.1)
- moved R113 174.6 mm to (62.9, 130.1)
- moved U101 174.6 mm to (73.1, 132.6)
- moved J118 147.8 mm to (186.0, 124.0)
- moved D107 121.8 mm to (120.6, 77.9), turned to 180 degrees
- moved D106 114.6 mm to (125.7, 77.9), turned to 180 degrees
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Connections:
- J115 pad 1: GND -> Gate1
- J115 pad 10: LED-CV2 -> LED2
- J115 pad 11: LED-CV1 -> LED1
- J115 pad 2: A2 -> Gate2
- J115 pad 3: A1 -> Net-(J115-Pad3)
- J115 pad 4: Btn -> LED_LFO
- J115 pad 5: LED_LFO -> LED-CV2
- J115 pad 6: LED4 -> LED-CV1
- J115 pad 7: LED3 -> LED-MIDI
- J115 pad 8: LED2 -> LED4
- J115 pad 9: LED1 -> LED3
- J116 pad 1: GND -> Gate1
- J116 pad 10: LED-CV2 -> LED2
- J116 pad 11: LED-CV1 -> LED1
- J116 pad 2: A2 -> Gate2
- J116 pad 3: A1 -> Net-(J115-Pad3)
- J116 pad 4: Btn -> LED_LFO
- J116 pad 5: LED_LFO -> LED-CV2
- J116 pad 6: LED4 -> LED-CV1
- J116 pad 7: LED3 -> LED-MIDI
- J116 pad 8: LED2 -> LED4
- J116 pad 9: LED1 -> LED3
- J117 pad 3: SCL -> Btn
- J117 pad 4: SDA -> A1
- J117 pad 5: Gate1 -> A2
- J117 pad 6: Gate2 -> SDA
- J117 pad 7: +5V -> SCL
- J117 pad 8: +12V -> +5V
- J118 pad 3: SCL -> Btn
- J118 pad 4: SDA -> A1
- J118 pad 5: Gate1 -> A2
- J118 pad 6: Gate2 -> SDA
- J118 pad 7: +5V -> SCL
- J118 pad 8: +12V -> +5V
