File: Kicad-Midi2CV2.sch (KiCad schematic (older format))
At the start: 101 parts, among them IC101 MCP4725module, IC102 MCP4725module, J101 Doepfer connector, J102 Vin 7-12v, J103 MIDI OUT, J104 Power Conn, J105 CV7 in, J106 Gate1, J107 MIDI IN, J108 CV6 in, J109 Gate2, J110 CV3 in, J111 Gate3, J112 CV1, J113 Gate4, J114 CV2, J115 ControlConn, J116 ControlConn, J117 I2C_Conn, J118 I2C_Conn, Q101 MMBT2222A, Q102 MMBT2222A, SW101 KY40_Rotary_Encoder_Module, U101 TL072, U102 TL072, U103 EL814

Commit message: Sch and PCB advancements
Parts:
- removed R118, R119: 10k, Resistor_SMD:R_0805_2012Metric_Pad1.15x1.40mm_HandSolder, symbol Device:R
- removed SW101: KY40_Rotary_Encoder_Module, Rotary_Encoder:KY-40-rotary-encoder-board, symbol Module:KY40_Rotary_Encoder_Module
- removed unit 2 of U102
- added C115, C116, C117, C118: 100n, Capacitor_SMD:C_0805_2012Metric_Pad1.15x1.40mm_HandSolder, symbol Device:C
- added R121, R122, R126, R127, R136, R137, R142, R143: 10k, Resistor_SMD:R_0805_2012Metric_Pad1.15x1.40mm_HandSolder, symbol Device:R
- added SW101: Rotary_Encoder_Switch, Rotary_Encoder:RotaryEncoder_Alps_EC11E-Switch_Vertical_H20mm, symbol Device:Rotary_Encoder_Switch
- added unit 1 of U102
- C119: renamed from C115; value 10n -> 47n
- J116: footprint Connector_PinHeader_2.54mm:PinHeader_1x11_P2.54mm_Horizontal -> Connector_PinHeader_2.54mm:PinHeader_1x11_P2.54mm_Vertical
- J118: footprint Connector_PinHeader_2.54mm:PinHeader_1x09_P2.54mm_Horizontal -> Connector_PinHeader_2.54mm:PinHeader_1x09_P2.54mm_Vertical
- renumbered C117 to C120, C116 to C121, R120 to R118, R121 to R119, R122 to R120, R126 to R128, R127 to R129, R128 to R133, R129 to R134, R133 to R135, R134 to R138, R135 to R139, R136 to R140, R137 to R141, R138 to R144
Connections:
- wire segments 410 -> 439
Other:
- moved on the sheet: C114, C120, C121, J104, R133, R134

Commit message: RC output on CV
Parts:
- added C114, C115: 47n, Capacitor_SMD:C_0805_2012Metric_Pad1.15x1.40mm_HandSolder, symbol Device:C
- added R108, R118: 100R, Resistor_SMD:R_0805_2012Metric_Pad1.15x1.40mm_HandSolder, symbol Device:R
- renumbered C114 to C116, C115 to C117, C116 to C118, C117 to C119, C118 to C120, C119 to C121, C120 to C122, C121 to C123, R108 to R109, R109 to R110, R110 to R111, R111 to R112, R112 to R113, R113 to R114, R114 to R115, R115 to R116, R116 to R117, R117 to R119, R118 to R120, R119 to R121, R120 to R122, R121 to R123, R122 to R124, R123 to R125, R124 to R126, R125 to R127, R126 to R128, R127 to R129, R128 to R130, R129 to R131, R130 to R132, R131 to R133, R132 to R134, R133 to R135, R134 to R136, R135 to R137, R136 to R138, R137 to R139, R138 to R140, R139 to R141, R140 to R142, R141 to R143, R142 to R144, R143 to R145, R144 to R146
Connections:
- wire segments 439 -> 447
Other:
- moved on the sheet: R104, R105, R113, R114, RV101, RV102, U101A, U101B
