File: Kicad-Midi2CV2.sch (KiCad schematic (older format))
At the start: 115 parts, among them IC101 MCP4725module, IC102 MCP4725module, J101 Doepfer connector, J102 Vin 7-12v, J103 MIDI OUT, J104 Power Conn, J105 CV7 in, J106 Gate1, J107 MIDI IN, J108 CV6 in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

Commit message: Component replacement
Parts:
- added H101, H102: 2,5mm, MountingHole:MountingHole_2.5mm_Pad_Via, symbol Mechanical:MountingHole
- added H103: 2,2mm, MountingHole:MountingHole_2.5mm_Pad_Via, symbol Mechanical:MountingHole
- added H104: 2,2mm, MountingHole:MountingHole_2.2mm_M2_Pad_Via, symbol Mechanical:MountingHole
- C114: value 47n -> 11n
- C115: value 47n -> 22n
- C117, C118: value 100n -> 33n
- C119, C120: value 100n -> 44n
- R104, R105: value 10k -> 11k
- R108: value 100R -> 110R
- R113, R114: value 10k -> 22k
- R118: value 100R -> 220R
- R123, R124, R128, R129: value 10k -> 33k
- R135, R136, R138, R139: value 10k -> 44k
Changed lines of the file:
@@
 P 9050 975
 F 0 "R104" V 8843 975 50  0000 C CNN
-F 1 "10k" V 8934 975 50  0000 C CNN
+F 1 "11k" V 8934 975 50  0000 C CNN
 F 2 "Resistor_SMD:R_0805_2012Metric_Pad1.15x1.40mm_HandSolder" V 8980 975 50  0001 C CNN
 F 3 "~" H 9050 975 50  0001 C CNN
@@
 P 9100 2150
 F 0 "R113" V 8893 2150 50  0000 C CNN
-F 1 "10k" V 8984 2150 50  0000 C CNN
+F 1 "22k" V 8984 2150 50  0000 C CNN
 F 2 "Resistor_SMD:R_0805_2012Metric_Pad1.15x1.40mm_HandSolder" V 9030 2150 50  0001 C CNN
 F 3 "~" H 9100 2150 50  0001 C CNN
@@
 P 9550 2150
 F 0 "R114" V 9343 2150 50  0000 C CNN
-F 1 "10k" V 9434 2150 50  0000 C CNN
+F 1 "22k" V 9434 2150 50  0000 C CNN
 F 2 "Resistor_SMD:R_0805_2012Metric_Pad1.15x1.40mm_HandSolder" V 9480 2150 50  0001 C CNN
 F 3 "~" H 9550 2150 50  0001 C CNN
@@
 P 9500 975
 F 0 "R105" V 9293 975 50  0000 C CNN
-F 1 "10k" V 9384 975 50  0000 C CNN
+F 1 "11k" V 9384 975 50  0000 C CNN
 F 2 "Resistor_SMD:R_0805_2012Metric_Pad1.15x1.40mm_HandSolder" V 9430 975 50  0001 C CNN
 F 3 "~" H 9500 975 50  0001 C CNN
@@
 P 9750 5450
 F 0 "R135" V 9543 5450 50  0000 C CNN
-F 1 "10k" V 9634 5450 50  0000 C CNN
+F 1 "44k" V 9634 5450 50  0000 C CNN
 F 2 "Resistor_SMD:R_0805_2012Metric_Pad1.15x1.40mm_HandSolder" V 9680 5450 50  0001 C CNN
 F 3 "~" H 9750 5450 50  0001 C CNN
@@
 P 10200 5450
 F 0 "R136" V 9993 5450 50  0000 C CNN
-F 1 "10k" V 10084 5450 50  0000 C CNN
+F 1 "44k" V 10084 5450 50  0000 C CNN
 F 2 "Resistor_SMD:R_0805_2012Metric_Pad1.15x1.40mm_HandSolder" V 10130 5450 50  0001 C CNN
 F 3 "~" H 10200 5450 50  0001 C CNN
@@
 P 9925 6050
 F 0 "C120" H 9825 6200 50  0000 L CNN
-F 1 "100n" H 9825 6300 50  0000 L CNN
+F 1 "44n" H 9825 6300 50  0000 L CNN
 F 2 "Capacitor_SMD:C_0805_2012Metric_Pad1.15x1.40mm_HandSolder" H 9963 5900 50  0001 C CNN
 F 3 "~" H 9925 6050 50  0001 C CNN
@@
 P 9175 5850
 F 0 "R138" V 8968 5850 50  0000 C CNN
-F 1 "10k" V 9059 5850 50  0000 C CNN
+F 1 "44k" V 9059 5850 50  0000 C CNN
 F 2 "Resistor_SMD:R_0805_2012Metric_Pad1.15x1.40mm_HandSolder" V 9105 5850 50  0001 C CNN
 F 3 "~" H 9175 5850 50  0001 C CNN
@@
 P 9650 5850
 F 0 "R139" V 9443 5850 50  0000 C CNN
-F 1 "10k" V 9534 5850 50  0000 C CNN
+F 1 "44k" V 9534 5850 50  0000 C CNN
 F 2 "Resistor_SMD:R_0805_2012Metric_Pad1.15x1.40mm_HandSolder" V 9580 5850 50  0001 C CNN
 F 3 "~" H 9650 5850 50  0001 C CNN
@@
 P 10025 5175
 F 0 "C119" H 9925 5325 50  0000 L CNN
-F 1 "100n" H 9925 5425 50  0000 L CNN
+F 1 "44n" H 9925 5425 50  0000 L CNN
 F 2 "Capacitor_SMD:C_0805_2012Metric_Pad1.15x1.40mm_HandSolder" H 10063 5025 50  0001 C CNN
 F 3 "~" H 10025 5175 50  0001 C CNN
@@
 P 9750 3925
 F 0 "R123" V 9543 3925 50  0000 C CNN
-F 1 "10k" V 9634 3925 50  0000 C CNN
+F 1 "33k" V 9634 3925 50  0000 C CNN
 F 2 "Resistor_SMD:R_0805_2012Metric_Pad1.15x1.40mm_HandSolder" V 9680 3925 50  0001 C CNN
 F 3 "~" H 9750 3925 50  0001 C CNN
@@
 P 10200 3925
 F 0 "R124" V 9993 3925 50  0000 C CNN
-F 1 "10k" V 10084 3925 50  0000 C CNN
+F 1 "33k" V 10084 3925 50  0000 C CNN
 F 2 "Resistor_SMD:R_0805_2012Metric_Pad1.15x1.40mm_HandSolder" V 10130 3925 50  0001 C CNN
 F 3 "~" H 10200 3925 50  0001 C CNN
@@
 P 9925 4525
 F 0 "C118" H 9825 4675 50  0000 L CNN
-F 1 "100n" H 9825 4775 50  0000 L CNN
+F 1 "33n" H 9825 4775 50  0000 L CNN
 F 2 "Capacitor_SMD:C_0805_2012Metric_Pad1.15x1.40mm_HandSolder" H 9963 4375 50  0001 C CNN
 F 3 "~" H 9925 4525 50  0001 C CNN
@@
 P 9175 4325
 F 0 "R128" V 8968 4325 50  0000 C CNN
-F 1 "10k" V 9059 4325 50  0000 C CNN
+F 1 "33k" V 9059 4325 50  0000 C CNN
 F 2 "Resistor_SMD:R_0805_2012Metric_Pad1.15x1.40mm_HandSolder" V 9105 4325 50  0001 C CNN
 F 3 "~" H 9175 4325 50  0001 C CNN
@@
 P 9650 4325
 F 0 "R129" V 9443 4325 50  0000 C CNN
-F 1 "10k" V 9534 4325 50  0000 C CNN
+F 1 "33k" V 9534 4325 50  0000 C CNN
 F 2 "Resistor_SMD:R_0805_2012Metric_Pad1.15x1.40mm_HandSolder" V 9580 4325 50  0001 C CNN
 F 3 "~" H 9650 4325 50  0001 C CNN
@@
 P 10025 3650
 F 0 "C117" H 9925 3800 50  0000 L CNN
-F 1 "100n" H 9925 3900 50  0000 L CNN
+F 1 "33n" H 9925 3900 50  0000 L CNN
 F 2 "Capacitor_SMD:C_0805_2012Metric_Pad1.15x1.40mm_HandSolder" H 10063 3500 50  0001 C CNN
 F 3 "~" H 10025 3650 50  0001 C CNN
@@
 P 10500 1525
 F 0 "R108" V 10293 1525 50  0000 C CNN
-F 1 "100R" V 10384 1525 50  0000 C CNN
+F 1 "110R" V 10384 1525 50  0000 C CNN
 F 2 "Resistor_SMD:R_0805_2012Metric_Pad1.15x1.40mm_HandSolder" V 10430 1525 50  0001 C CNN
 F 3 "~" H 10500 1525 50  0001 C CNN
@@
 P 10475 2700
 F 0 "R118" V 10268 2700 50  0000 C CNN
-F 1 "100R" V 10359 2700 50  0000 C CNN
+F 1 "220R" V 10359 2700 50  0000 C CNN
 F 2 "Resistor_SMD:R_0805_2012Metric_Pad1.15x1.40mm_HandSolder" V 10405 2700 50  0001 C CNN
 F 3 "~" H 10475 2700 50  0001 C CNN
@@
 P 10675 2875
 F 0 "C115" H 10575 3025 50  0000 L CNN
-F 1 "47n" H 10575 3125 50  0000 L CNN
+F 1 "22n" H 10575 3125 50  0000 L CNN
 F 2 "Capacitor_SMD:C_0805_2012Metric_Pad1.15x1.40mm_HandSolder" H 10713 2725 50  0001 C CNN
 F 3 "~" H 10675 2875 50  0001 C CNN
@@
 P 10675 1675
 F 0 "C114" H 10575 1825 50  0000 L CNN
-F 1 "47n" H 10575 1925 50  0000 L CNN
+F 1 "11n" H 10575 1925 50  0000 L CNN
 F 2 "Capacitor_SMD:C_0805_2012Metric_Pad1.15x1.40mm_HandSolder" H 10713 1525 50  0001 C CNN
 F 3 "~" H 10675 1675 50  0001 C CNN
@@
 	6550 5100 6550 5300
 Connection ~ 6550 5100
+$Comp
+L Mechanical:MountingHole H101
+U 1 1 5D3AEF13
+P 7775 6150
+F 0 "H101" H 7875 6196 50  0000 L CNN
+F 1 "2,5mm" H 7875 6105 50  0000 L CNN
+F 2 "MountingHole:MountingHole_2.5mm_Pad_Via" H 7775 6150 50  0001 C CNN
+F 3 "~" H 7775 6150 50  0001 C CNN
+	1    7775 6150
+	1    0    0    -1
+$EndComp
+$Comp
+L Mechanical:MountingHole H102
+U 1 1 5D3AF3EC
+P 8225 6150
+F 0 "H102" H 8325 6196 50  0000 L CNN
+F 1 "2,5mm" H 8325 6105 50  0000 L CNN
+F 2 "MountingHole:MountingHole_2.5mm_Pad_Via" H 8225 6150 50  0001 C CNN
+F 3 "~" H 8225 6150 50  0001 C CNN
+	1    8225 6150
+	1    0    0    -1
+$EndComp
+$Comp
+L Mechanical:MountingHole H104
+U 1 1 5D3AF4F8
+P 8225 6350
+F 0 "H104" H 8325 6396 50  0000 L CNN
+F 1 "2,2mm" H 8325 6305 50  0000 L CNN
+F 2 "MountingHole:MountingHole_2.2mm_M2_Pad_Via" H 8225 6350 50  0001 C CNN
+F 3 "~" H 8225 6350 50  0001 C CNN
+	1    8225 6350
+	1    0    0    -1
+$EndComp
+$Comp
+L Mechanical:MountingHole H103
+U 1 1 5D3AF63A
+P 7775 6350
+F 0 "H103" H 7875 6396 50  0000 L CNN
+F 1 "2,2mm" H 7875 6305 50  0000 L CNN
+F 2 "MountingHole:MountingHole_2.5mm_Pad_Via" H 7775 6350 50  0001 C CNN
+F 3 "~" H 7775 6350 50  0001 C CNN
+	1    7775 6350
+	1    0    0    -1
+$EndComp
+$Comp
+L power:GND #PWR?
+U 1 1 5D3B40A8
+P 7850 5000
+F 0 "#PWR?" H 7850 4750 50  0001 C CNN
+F 1 "GND" H 7855 4827 50  0000 C CNN
+F 2 "" H 7850 5000 50  0001 C CNN
+F 3 "" H 7850 5000 50  0001 C CNN
+	1    7850 5000
+	1    0    0    -1
+$EndComp
 $EndSCHEMATC

Commit message: Routing....
Changed lines of the file:
@@
 Text GLabel 2400 5975 2    50   Input ~ 0
 LED-MIDI
-Text GLabel 4325 6525 0    50   Input ~ 0
+Text GLabel 4325 7225 0    50   Input ~ 0
 LED1
-Text GLabel 4325 6625 0    50   Input ~ 0
+Text GLabel 4325 7325 0    50   Input ~ 0
 LED2
-Text GLabel 4325 6725 0    50   Input ~ 0
+Text GLabel 4325 7425 0    50   Input ~ 0
 LED3
-Text GLabel 4325 6825 0    50   Input ~ 0
+Text GLabel 4325 7525 0    50   Input ~ 0
 LED4
 $Comp
@@
 Wire Wire Line
 	1150 7600 1300 7600
-Text GLabel 4325 7525 0    50   Input ~ 0
+Text GLabel 4325 7025 0    50   Input ~ 0
 Gate1
-Text GLabel 4325 7425 0    50   Input ~ 0
+Text GLabel 4325 7125 0    50   Input ~ 0
 Gate2
 Text GLabel 5350 4800 2    50   Input ~ 0
@@
 Wire Notes Line
 	6300 500  8525 500
-Text GLabel 4325 7125 0    50   Input ~ 0
+Text GLabel 4325 6825 0    50   Input ~ 0
 LED-CV2
-Text GLabel 4325 7025 0    50   Input ~ 0
+Text GLabel 4325 6625 0    50   Input ~ 0
 LED-CV1
-Text GLabel 4325 6925 0    50   Input ~ 0
+Text GLabel 4325 6725 0    50   Input ~ 0
 LED-MIDI
 Wire Notes Line
@@
 L power:GND #PWR0128
 U 1 1 5CAA25A2
-P 3875 7350
-F 0 "#PWR0128" H 3875 7100 50  0001 C CNN
-F 1 "GND" H 3880 7177 50  0000 C CNN
-F 2 "" H 3875 7350 50  0001 C CNN
-F 3 "" H 3875 7350 50  0001 C CNN
-	1    3875 7350
+P 3900 6950
+F 0 "#PWR0128" H 3900 6700 50  0001 C CNN
+F 1 "GND" H 3905 6777 50  0000 C CNN
+F 2 "" H 3900 6950 50  0001 C CNN
+F 3 "" H 3900 6950 50  0001 C CNN
+	1    3900 6950
 	1    0    0    -1
 $EndComp
@@
 	4325 6825 4400 6825
 Wire Wire Line
-	4325 6925 4400 6925
-Wire Wire Line
 	4325 7025 4400 7025
 Wire Wire Line
@@
 Wire Wire Line
 	4325 7425 4400 7425
-Wire Wire Line
-	3775 7275 3775 7300
 Wire Wire Line
 	4475 7225 4400 7225
@@
 Wire Wire Line
 	4400 7250 4400 7325
-Connection ~ 4400 7325
 Wire Wire Line
 	4400 7325 4475 7325
@@
 Wire Wire Line
 	2575 900  3050 900
-Text GLabel 4325 7225 0    50   Input ~ 0
+Text GLabel 4325 6525 0    50   Input ~ 0
 LED_LFO
 Wire Wire Line
@@
 Connection ~ 6000 7475
 Wire Wire Line
-	3875 7325 4400 7325
-Wire Wire Line
 	4325 7525 4400 7525
 Connection ~ 4400 7525
@@
 $EndComp
 $Comp
-L power:GND #PWR?
+L power:GND #PWR0131
 U 1 1 5D3B40A8
 P 7850 5000
-F 0 "#PWR?" H 7850 4750 50  0001 C CNN
+F 0 "#PWR0131" H 7850 4750 50  0001 C CNN
 F 1 "GND" H 7855 4827 50  0000 C CNN
 F 2 "" H 7850 5000 50  0001 C CNN
@@
 	1    0    0    -1
 $EndComp
+Wire Wire Line
+	3900 6925 3900 6950
+Wire Wire Line
+	3900 6925 4400 6925
+Wire Wire Line
+	4325 7325 4400 7325
+Connection ~ 4400 7325
 $EndSCHEMATC

Commit message: Initial PCB finished - no DRC
Parts:
- added R147: 133R, Resistor_SMD:R_0805_2012Metric_Pad1.15x1.40mm_HandSolder, symbol Device:R
- added R148: 144R, Resistor_SMD:R_0805_2012Metric_Pad1.15x1.40mm_HandSolder, symbol Device:R
- JP104: value GND MIDI OUT -> GND MIDI IN
Connections:
- wire segments 447 -> 449
Changed lines of the file:
@@
 P 1375 4300
 F 0 "JP104" H 1175 4425 50  0000 L CNN
-F 1 "GND MIDI OUT" H 1420 4426 50  0000 L CNN
+F 1 "GND MIDI IN" H 1420 4426 50  0000 L CNN
 F 2 "Jumper:SolderJumper-2_P1.3mm_Open_RoundedPad1.0x1.5mm" H 1375 4300 50  0001 C CNN
 F 3 "~" H 1375 4300 50  0001 C CNN
@@
 	1    0    0    1
 $EndComp
-Text GLabel 10775 4225 2    50   Input ~ 0
+Text GLabel 11100 4250 3    50   Input ~ 0
 Gate3Gain
-Text GLabel 10775 5750 2    50   Input ~ 0
+Text GLabel 11125 5800 3    50   Input ~ 0
 Gate4Gain
 $Comp
@@
 Wire Wire Line
 	8975 4325 9025 4325
-Wire Wire Line
-	10700 4225 10775 4225
-Wire Wire Line
-	10700 3650 10700 3925
-Wire Wire Line
-	10175 3650 10700 3650
-Wire Wire Line
-	10350 3925 10700 3925
-Connection ~ 10700 3925
-Wire Wire Line
-	10700 3925 10700 4225
-Wire Wire Line
-	10650 4225 10700 4225
-Connection ~ 10700 4225
-Wire Wire Line
-	10700 5175 10700 5450
-Wire Wire Line
-	10175 5175 10700 5175
-Wire Wire Line
-	10350 5450 10700 5450
-Connection ~ 10700 5450
-Wire Wire Line
-	10700 5450 10700 5750
-Wire Wire Line
-	10650 5750 10700 5750
-Connection ~ 10700 5750
-Wire Wire Line
-	10700 5750 10775 5750
 $Comp
 L Device:R R108
@@
 	4325 7325 4400 7325
 Connection ~ 4400 7325
+$Comp
+L Device:R R147
+U 1 1 5D6DD7CC
+P 10925 4225
+F 0 "R147" V 10718 4225 50  0000 C CNN
+F 1 "133R" V 10809 4225 50  0000 C CNN
+F 2 "Resistor_SMD:R_0805_2012Metric_Pad1.15x1.40mm_HandSolder" V 10855 4225 50  0001 C CNN
+F 3 "~" H 10925 4225 50  0001 C CNN
+	1    10925 4225
+	0    1    1    0
+$EndComp
+Wire Wire Line
+	11075 4225 11100 4225
+Wire Wire Line
+	11100 4225 11100 4250
+$Comp
+L Device:R R148
+U 1 1 5D718073
+P 10925 5750
+F 0 "R148" V 10718 5750 50  0000 C CNN
+F 1 "144R" V 10809 5750 50  0000 C CNN
+F 2 "Resistor_SMD:R_0805_2012Metric_Pad1.15x1.40mm_HandSolder" V 10855 5750 50  0001 C CNN
+F 3 "~" H 10925 5750 50  0001 C CNN
+	1    10925 5750
+	0    1    1    0
+$EndComp
+Wire Wire Line
+	11075 5750 11125 5750
+Wire Wire Line
+	11125 5750 11125 5800
+Wire Wire Line
+	10650 5750 10775 5750
+Wire Wire Line
+	11125 5450 11125 5750
+Connection ~ 11125 5750
+Wire Wire Line
+	10350 5450 11125 5450
+Wire Wire Line
+	11125 5175 11125 5450
+Wire Wire Line
+	10175 5175 11125 5175
+Connection ~ 11125 5450
+Wire Wire Line
+	10650 4225 10775 4225
+Wire Wire Line
+	11100 3650 11100 3925
+Connection ~ 11100 4225
+Connection ~ 11100 3925
+Wire Wire Line
+	11100 3925 11100 4225
+Wire Wire Line
+	10175 3650 11100 3650
+Wire Wire Line
+	10350 3925 11100 3925
 $EndSCHEMATC

Commit message: MOVED PINS AROUND ON ARDUINO
Parts:
- IC101, IC102: symbol aj_adc_dac:MCP4725module -> Kicad-Midi2CV2-rescue:MCP4725module-aj_adc_dac
Changed lines of the file:
@@
 $EndComp
 $Comp
-L aj_adc_dac:MCP4725module IC102
+L Kicad-Midi2CV2-rescue:MCP4725module-aj_adc_dac IC102
 U 1 1 5C1C16C6
 P 7300 2400
@@
 $EndComp
 $Comp
-L aj_adc_dac:MCP4725module IC101
+L Kicad-Midi2CV2-rescue:MCP4725module-aj_adc_dac IC101
 U 1 1 5C1C326B
 P 7300 1350
@@
 Text GLabel 3950 4200 0    50   Input ~ 0
 Gate1
-Text GLabel 3950 4300 0    50   Input ~ 0
+Text GLabel 3950 4500 0    50   Input ~ 0
 Gate2
 Text GLabel 5350 4200 2    50   Input ~ 0
 Btn
-Text GLabel 3950 4700 0    50   Input ~ 0
+Text GLabel 3950 4400 0    50   Input ~ 0
 LED-CV1
 Wire Wire Line
@@
 Text Label 3550 3600 0    50   ~ 0
 RX
-Text GLabel 3950 4400 0    50   Input ~ 0
+Text GLabel 3950 4600 0    50   Input ~ 0
 Gate3
-Text GLabel 3950 4500 0    50   Input ~ 0
+Text GLabel 3950 4700 0    50   Input ~ 0
 Gate4
 Wire Wire Line
@@
 Wire Wire Line
 	950  6300 750  6300
-Text GLabel 3950 4600 0    50   Input ~ 0
+Text GLabel 3950 4300 0    50   Input ~ 0
 LED-MIDI
 Wire Wire Line
